Commit message: Update robot description to not root into world and root frames
This will help when connecting the kinova arm to the dingo virtually

File: kinova_description/urdf/j2n6s300_standalone.xacro (robot description, xacro)
@@ -15,13 +15,4 @@
 	xmlns:xacro="http://www.ros.org/wiki/xacro" name="j2n6s300">
   <xacro:include filename="$(find kinova_description)/urdf/j2n6s300.xacro"/>
-  <link name="root"/>
-  <!-- for gazebo -->
-  <link name="world"/>
-  <joint name="connect_root_and_world" type="fixed">
-    <child link="root" />
-    <parent link="world" />
-    <origin xyz="0 0 0" rpy="0 0 0" />
-  </joint>
-  <xacro:property name="robot_root" value="root" />
-  <xacro:j2n6s300  base_parent="${robot_root}"/>
+  <xacro:j2n6s300  base_parent="arm_mount"/>
 </robot>

Commit message: Ensure arm_mount is a valid link

File: kinova_description/urdf/j2n6s300_standalone.xacro (robot description, xacro)
@@ -15,4 +15,5 @@
 	xmlns:xacro="http://www.ros.org/wiki/xacro" name="j2n6s300">
   <xacro:include filename="$(find kinova_description)/urdf/j2n6s300.xacro"/>
+  <link name="arm_mount" />
   <xacro:j2n6s300  base_parent="arm_mount"/>
 </robot>
